Commit message: added gazebo simulation for camera

File: src/carbot_hardware/description/urdf/bigbrain.urdf.xacro (robot description, xacro)
@@ -4,5 +4,5 @@
   <!-- Constants for robot dimensions -->
   <xacro:property name="PI" value="3.1415926535897931"/>
-  <xacro:property name="base_mass" value="100.0" /> <!-- arbitrary value for base mass -->
+  <xacro:property name="base_mass" value="10" /> <!-- arbitrary value for base mass -->
   <xacro:property name="base_width" value="0.1351" />
   <xacro:property name="base_length" value="0.1778" />
@@ -13,5 +13,6 @@
   <xacro:property name="wheel_radius" value="0.0375" />
   <xacro:property name="wheeltrack" value=".1651"/>
-  <xacro:property name="friction" value="2"/>
+  <xacro:property name="friction" value="3"/>
+  <xacro:property name="damping" value="0.01"/>
   <!-- ======================================================================================== -->
   <!-- Base Link -->
@@ -49,5 +50,5 @@
       <origin xyz="0 0 ${base_height/2 + wheel_radius}" rpy="0 0 0"/>
       <axis xyz="0 0 1"/>
-      <dynamics damping="0.2"/>
+      <dynamics damping="${damping}"/>
     </joint>
     <!-- ==================================================================== -->
@@ -93,5 +94,5 @@
             <axis xyz="1 0 0"/>
             <limit effort="1000.0" velocity="100.0"/>
-            <dynamics damping="0.2"/>
+            <dynamics damping="${damping}"/>
             <mimic joint="${prefix}virtual_rear_wheel_joint" multiplier="1.0" offset="0.0"/>
         </joint>
@@ -149,5 +150,5 @@
             <axis xyz="1 0 0"/>
             <limit effort="100.0" velocity="100.0"/>
-            <dynamics damping="0.2"/>
+            <dynamics damping="${damping}"/>
             <mimic joint="${prefix}virtual_rear_wheel_joint" multiplier="1.0" offset="0.0"/>
         </joint>
@@ -157,6 +158,6 @@
             <origin xyz="${wheelbase/2} ${base_width/2 * direction} -${base_height/2}" rpy="0 0 ${PI/2}"/>
             <axis xyz="0 0 1"/>
-            <limit lower="-0.7" upper="0.7" effort="1000.0" velocity="0.0000001"/>
-            <dynamics damping="0.2"/>
+            <limit lower="-0.5" upper="0.5" effort="1000.0" velocity="0.0000001"/>
+            <dynamics damping="${damping}"/>
             <mimic joint="${prefix}virtual_front_wheel_joint" multiplier="1.0" offset="0.0"/>
         </joint>
@@ -194,5 +195,5 @@
       <axis xyz="1 0 0"/>
       <limit effort="100.0" velocity="100.0"/>
-      <dynamics damping="0.2"/>
+      <dynamics damping="${damping}"/>
     </joint>
     <link name="${prefix}virtual_front_wheel">
@@ -222,5 +223,5 @@
       <axis xyz="0 0 1"/>
       <limit lower="-0.4" upper="0.4" effort="100.0" velocity="100.0"/>
-      <dynamics damping="0.2"/>
+      <dynamics damping="${damping}"/>
     </joint>
   </xacro:macro>

File: src/carbot_hardware/description/urdf/carlikebot.urdf.xacro (robot description, xacro)
@@ -12,5 +12,8 @@
   <xacro:include filename="$(find carbot_hardware)/ros2_control/carlikebot.ros2_control.xacro" />
   <!-- <xacro:include filename="$(find carbot_hardware)/ros2_control/sim.xacro"/> -->
+  <!-- Import Camera -->
+  <xacro:include filename="$(find carbot_hardware)/urdf/camera.xacro" />
   <xacro:carlikebot prefix="$(arg prefix)" />
+  <xacro:camera prefix="$(arg prefix)"/>
   <xacro:carlikebot_ros2_control name="CarlikeBot" prefix="$(arg prefix)" />
 </robot>
