Commit message: added lidar

File: src/carbot_hardware/description/urdf/camera.xacro (robot description, xacro)
@@ -12,5 +12,5 @@
             <parent link="${prefix}chassis_link"/>
             <child link="${prefix}camera_link"/>
-            <origin xyz="${x_transform} ${y_transform} ${z_transform}" rpy="${r_transform} ${p_transform} ${y_transform}"/>
+            <origin xyz="${x_transform / 2} ${y_transform} ${z_transform}" rpy="${r_transform} ${p_transform} ${y_transform}"/>
         </joint>
         <link name="${prefix}camera_link">
@@ -46,5 +46,5 @@
                     </clip>
                 </camera>
-                <plugin name="laser_controller" filename="libgazebo_ros_camera.so">
+                <plugin name="camera_controller" filename="libgazebo_ros_camera.so">
                     <frame_name>camera_link_optical</frame_name>
                 </plugin>

File: src/carbot_hardware/description/urdf/carlikebot.urdf.xacro (robot description, xacro)
@@ -14,6 +14,9 @@
   <!-- Import Camera -->
   <xacro:include filename="$(find carbot_hardware)/urdf/camera.xacro" />
+  <!-- Import LiDAR -->
+  <xacro:include filename="$(find carbot_hardware)/urdf/lidar.xacro" />
   <xacro:carlikebot prefix="$(arg prefix)" />
   <xacro:camera prefix="$(arg prefix)"/>
+  <xacro:lidar prefix="$(arg prefix)"/>
   <xacro:carlikebot_ros2_control name="CarlikeBot" prefix="$(arg prefix)" />
 </robot>
