Commit message: changed effort to position and velocity

File: src/carbot_hardware/description/ros2_control/carlikebot.ros2_control.xacro (robot description, xacro)
@@ -17,10 +17,10 @@
         </hardware>
         <joint name="${prefix}virtual_rear_wheel_joint">
-          <command_interface name="effort"/>
+          <command_interface name="velocity"/>
           <state_interface name="velocity"/>
           <state_interface name="position"/>
         </joint>
         <joint name="${prefix}virtual_front_wheel_joint">
-          <command_interface name="effort"/>
+          <command_interface name="position"/>
           <state_interface name="position"/>
         </joint>
@@ -38,5 +38,5 @@
         <!-- drive joint -->
         <joint name="${prefix}virtual_rear_wheel_joint">
-          <command_interface name="effort">
+          <command_interface name="velocity">
             <param name="min">-1000</param>
             <param name="max">1000</param>
@@ -71,5 +71,5 @@
         <!-- steer joint -->
         <joint name="${prefix}virtual_front_wheel_joint">
-          <command_interface name="effort">
+          <command_interface name="position">
             <param name="min">-1000</param>
             <param name="max">1000</param>

File: src/carbot_hardware/description/urdf/bigbrain.urdf.xacro (robot description, xacro)
@@ -4,5 +4,5 @@
   <!-- Constants for robot dimensions -->
   <xacro:property name="PI" value="3.1415926535897931"/>
-  <xacro:property name="base_mass" value="4.0" /> <!-- arbitrary value for base mass -->
+  <xacro:property name="base_mass" value="100.0" /> <!-- arbitrary value for base mass -->
   <xacro:property name="base_width" value="0.1351" />
   <xacro:property name="base_length" value="0.1778" />
@@ -13,5 +13,5 @@
   <xacro:property name="wheel_radius" value="0.0375" />
   <xacro:property name="wheeltrack" value=".1651"/>
-  <xacro:property name="friction" value="1"/>
+  <xacro:property name="friction" value="2"/>
   <!-- ======================================================================================== -->
   <!-- Base Link -->
@@ -92,5 +92,5 @@
             <origin xyz="-${wheelbase/2} ${base_width/2 * direction} -${base_height/2}" rpy="0 0 ${PI/2}"/>
             <axis xyz="1 0 0"/>
-            <limit effort="100.0" velocity="100.0"/>
+            <limit effort="1000.0" velocity="100.0"/>
             <dynamics damping="0.2"/>
             <mimic joint="${prefix}virtual_rear_wheel_joint" multiplier="1.0" offset="0.0"/>
@@ -157,5 +157,5 @@
             <origin xyz="${wheelbase/2} ${base_width/2 * direction} -${base_height/2}" rpy="0 0 ${PI/2}"/>
             <axis xyz="0 0 1"/>
-            <limit lower="-0.4" upper="0.4" effort="100.0" velocity="100.0"/>
+            <limit lower="-0.7" upper="0.7" effort="1000.0" velocity="0.0000001"/>
             <dynamics damping="0.2"/>
             <mimic joint="${prefix}virtual_front_wheel_joint" multiplier="1.0" offset="0.0"/>

Commit message: dsadada

File: src/carbot_hardware/description/ros2_control/carlikebot.ros2_control.xacro (robot description, xacro)
@@ -2,4 +2,5 @@
 <robot xmlns:xacro="http://www.ros.org/wiki/xacro">
   <xacro:macro name="carlikebot_ros2_control" params="name prefix">
+  <xacro:property name="speed_multiplier" value="1"/>
     <xacro:unless value="$(arg sim_mode)">
       <ros2_control name="${name}" type="system">
@@ -62,5 +63,5 @@
         <joint name="${prefix}rear_left_wheel_joint">
           <param name="mimic">virtual_rear_wheel_joint</param>
-          <param name="multiplier">1</param>
+          <param name="multiplier">${speed_multiplier}</param>
           <state_interface name="velocity">
             <param name="initial_value">0.0</param>
@@ -75,5 +76,5 @@
         <joint name="${prefix}rear_right_wheel_joint">
           <param name="mimic">virtual_rear_wheel_joint</param>
-          <param name="multiplier">1</param>
+          <param name="multiplier">${speed_multiplier}</param>
           <state_interface name="velocity">
             <param name="initial_value">0.0</param>
@@ -101,5 +102,5 @@
         <joint name="${prefix}front_right_wheel_joint">
           <param name="mimic">virtual_rear_wheel_joint</param>
-          <param name="multiplier">1</param>
+          <param name="multiplier">${speed_multiplier}</param>
           <state_interface name="velocity">
             <param name="initial_value">0.0</param>
@@ -114,5 +115,5 @@
         <joint name="${prefix}front_left_wheel_joint">
           <param name="mimic">virtual_rear_wheel_joint</param>
-          <param name="multiplier">1</param>
+          <param name="multiplier">${speed_multiplier}</param>
           <state_interface name="velocity">
             <param name="initial_value">0.0</param>

File: src/carbot_hardware/description/urdf/bigbrain.urdf.xacro (robot description, xacro)
@@ -170,5 +170,5 @@
     <!-- virtual rear wheel -->
     <link name="${prefix}virtual_rear_wheel">
-      <visual>
+      <!-- <visual>
         <origin xyz="0 0 0" rpy="${PI/2} 0 ${PI/2}"/>
         <geometry>
@@ -176,5 +176,5 @@
         </geometry>
         <material name="invisible"/>
-      </visual>
+      </visual> -->
       <inertial>
         <origin xyz="0 0 0" rpy="${PI/2} 0 ${PI/2}"/>
@@ -198,5 +198,5 @@
     </joint>
     <link name="${prefix}virtual_front_wheel">
-      <visual>
+      <!-- <visual>
         <origin xyz="0 0 0" rpy="${PI/2} 0 ${PI/2}"/>
         <geometry>
@@ -204,5 +204,5 @@
         </geometry>
         <material name="invisible"/>
-      </visual>
+      </visual> -->
       <inertial>
         <origin xyz="0 0 0" rpy="${PI/2} 0 ${PI/2}"/>
