Commit message: Started working on URDF

File: ros2_ws/src/robot_hardware/description/urdf/core.urdf.xacro (robot description, xacro)
@@ -1,25 +1,25 @@
 <?xml version="1.0"?>
 <!-- 4 Wheel Robot with front steering and rear drive -->
-<robot xmlns:xacro="http://www.ros.org/wiki/xacro" name="carlikebot_robot">
+<robot xmlns:xacro="http://www.ros.org/wiki/xacro" name="robot_hardware">
   <xacro:arg name="prefix" default="" />
   <xacro:arg name="sim_mode" default="false"/>
   <!-- Import Constants -->
-  <xacro:include filename="$(find carbot_hardware)/urdf/util/constants.xacro" />
+  <xacro:include filename="$(find robot_hardware)/urdf/util/constants.xacro" />
   <!-- Import Robot Description -->
-  <xacro:include filename="$(find carbot_hardware)/urdf/robot.urdf.xacro" />
+  <xacro:include filename="$(find robot_hardware)/urdf/robot.urdf.xacro" />
   <!-- Import Rviz colors -->
-  <xacro:include filename="$(find carbot_hardware)/urdf/util/carlikebot.materials.xacro" />
+  <xacro:include filename="$(find robot_hardware)/urdf/util/materials.xacro" />
   <!-- Import Hardware Interface -->
-  <xacro:include filename="$(find carbot_hardware)/ros2_control/carlikebot.ros2_control.xacro" />
-  <!-- <xacro:include filename="$(find carbot_hardware)/ros2_control/sim.xacro"/> -->
+  <xacro:include filename="$(find robot_hardware)/ros2_control/robot_hardware.ros2_control.xacro" />
+  <!-- <xacro:include filename="$(find robot_hardware)/ros2_control/sim.xacro"/> -->
   <!-- Import Camera -->
-  <!-- <xacro:include filename="$(find carbot_hardware)/urdf/components/camera.xacro" /> -->
+  <!-- <xacro:include filename="$(find robot_hardware)/urdf/components/camera.xacro" /> -->
   <!-- Import Depth Camera -->
-  <!-- <xacro:include filename="$(find carbot_hardware)/urdf/components/depth_camera.xacro" /> -->
+  <!-- <xacro:include filename="$(find robot_hardware)/urdf/components/depth_camera.xacro" /> -->
   <!-- Import LiDAR -->
-  <xacro:include filename="$(find carbot_hardware)/urdf/components/lidar.xacro" />
-  <xacro:carlikebot prefix="$(arg prefix)" />
+  <!-- <xacro:include filename="$(find robot_hardware)/urdf/components/lidar.xacro" /> -->
+  <xacro:robot_hardware prefix="$(arg prefix)" />
   <!-- <xacro:camera prefix="$(arg prefix)"/> -->
-  <xacro:lidar prefix="$(arg prefix)"/>
-  <xacro:carlikebot_ros2_control name="CarlikeBot" prefix="$(arg prefix)" />
+  <!-- <xacro:lidar prefix="$(arg prefix)"/> -->
+  <xacro:robot_hardware_ros2_control name="RobotSystemHardware" prefix="$(arg prefix)" />
 </robot>

File: ros2_ws/src/robot_hardware/description/urdf/robot.urdf.xacro (robot description, xacro)
@@ -1,5 +1,5 @@
 <?xml version="1.0"?>
 <robot xmlns:xacro="http://www.ros.org/wiki/xacro">
-  <xacro:macro name="carlikebot" params="prefix">
+  <xacro:macro name="robot_hardware" params="prefix">
     <!-- Base Link -->
     <link name="${prefix}base_link"/>
@@ -9,5 +9,5 @@
         <origin xyz="0 0 0" rpy="0 0 ${PI/2}"/>
         <geometry>
-          <mesh filename="file://$(find carbot_hardware)/urdf/assets/Chassis.stl"/>
+          <mesh filename="file://$(find robot_hardware)/urdf/meshes/Chassis.stl"/>
         </geometry>
       </collision>
@@ -15,5 +15,6 @@
         <origin xyz="0 0 0" rpy="0 0 ${PI/2}"/>
         <geometry>
-          <mesh filename="file://$(find carbot_hardware)/urdf/assets/Chassis.stl"/>
+        <!-- <box size="1 1 1"/> -->
+        <mesh filename="package://robot_hardware/urdf/meshes/Chassis.stl"/>
         </geometry>
         <material name="grey"/>
@@ -45,5 +46,5 @@
                 <origin xyz="0 0 0" rpy="${side * -PI/2} 0 0"/>
                 <geometry>
-                  <mesh filename="file://$(find carbot_hardware)/urdf/assets/Wheel.stl"/>
+                  <mesh filename="file://$(find robot_hardware)/urdf/meshes/Wheel.stl"/>
                 </geometry>
                 <surface>
@@ -60,5 +61,5 @@
                   <origin xyz="0 0 0" rpy="${side * -PI/2} 0 0"/>
                   <geometry>
-                      <mesh filename="file://$(find carbot_hardware)/urdf/assets/Wheel.stl"/>
+                      <mesh filename="file://$(find robot_hardware)/urdf/meshes/Wheel.stl"/>
                   </geometry>
                   <material name="black"/>
