Commit message: fixed Rviz default path

File: ros2_ws/src/robot_hardware/description/urdf/robot.urdf.xacro (robot description, xacro)
@@ -7,5 +7,5 @@
     <link name="${prefix}chassis_link">
       <collision>
-        <origin xyz="0 0 0" rpy="0 0 ${PI/2}"/>
+        <origin xyz="0 0 0" rpy="0 0 0"/>
         <geometry>
           <mesh filename="file://$(find robot_hardware)/urdf/meshes/Chassis.stl"/>
@@ -13,10 +13,11 @@
       </collision>
       <visual>
-        <origin xyz="0 0 0" rpy="0 0 ${PI/2}"/>
+        <origin xyz="0 0 0" rpy="0 0 0"/>
         <geometry>
         <!-- <box size="1 1 1"/> -->
         <mesh filename="package://robot_hardware/urdf/meshes/Chassis.stl"/>
         </geometry>
-        <material name="grey"/>
+        <cast_shadows>true</cast_shadows>
+        <!-- <material name="grey"/> -->
       </visual>
       <inertial>
@@ -30,10 +31,10 @@
     </link>
       <gazebo reference="chassis_link">
-        <material>Gazebo/Grey</material>
+        <!-- <material>Gazebo/Grey</material> -->
       </gazebo>
       <joint name="${prefix}chassis_joint" type="fixed">
         <parent link="${prefix}base_link"/>
         <child link="${prefix}chassis_link"/>
-        <origin xyz="0 0 ${.0199 + wheel_radius}" rpy="0 0 0"/>
+        <origin xyz="0 0 0" rpy="0 0 0"/>
         <axis xyz="0 0 1"/>
         <dynamics damping="${damping}"/>

Commit message: Fixed URDF to have proper steering

File: ros2_ws/src/robot_hardware/description/urdf/robot.urdf.xacro (robot description, xacro)
@@ -2,96 +2,14 @@
 <robot xmlns:xacro="http://www.ros.org/wiki/xacro">
   <xacro:macro name="robot_hardware" params="prefix">
-    <!-- Base Link -->
-    <link name="${prefix}base_link"/>
-    <!-- Chassis -->
-    <link name="${prefix}chassis_link">
-      <collision>
-        <origin xyz="0 0 0" rpy="0 0 0"/>
-        <geometry>
-          <mesh filename="file://$(find robot_hardware)/urdf/meshes/Chassis.stl"/>
-        </geometry>
-      </collision>
-      <visual>
-        <origin xyz="0 0 0" rpy="0 0 0"/>
-        <geometry>
-        <!-- <box size="1 1 1"/> -->
-        <mesh filename="package://robot_hardware/urdf/meshes/Chassis.stl"/>
-        </geometry>
-        <cast_shadows>true</cast_shadows>
-        <!-- <material name="grey"/> -->
-      </visual>
-      <inertial>
-        <origin xyz="0 0 0" rpy="0 0 0"/>
-        <mass value="${base_mass}"/>
-          <inertia
-            ixx="0.000270" ixy="0.0" ixz="0.0"
-            iyy="0.000270" iyz="0.0"
-            izz="0.000426"/>
-        </inertial>
-    </link>
-      <gazebo reference="chassis_link">
-        <!-- <material>Gazebo/Grey</material> -->
-      </gazebo>
-      <joint name="${prefix}chassis_joint" type="fixed">
-        <parent link="${prefix}base_link"/>
-        <child link="${prefix}chassis_link"/>
-        <origin xyz="0 0 0" rpy="0 0 0"/>
-        <axis xyz="0 0 1"/>
-        <dynamics damping="${damping}"/>
-      </joint>
-      <!-- ==================================================================== -->
-      <xacro:macro name="wheel" params="name x y z front side">
-          <link name="${name}_wheel">
-              <!-- COLLISION -->
-              <collision>
-                <origin xyz="0 0 0" rpy="${side * -PI/2} 0 0"/>
-                <geometry>
-                  <mesh filename="file://$(find robot_hardware)/urdf/meshes/Wheel.stl"/>
-                </geometry>
-                <surface>
-                    <friction>
-                      <ode>
-                        <mu value="${friction}"/>
-                        <mu2 value="${friction}"/>
-                      </ode>
-                    </friction>
-                  </surface>
-              </collision>
-              <!-- VISIUAL -->
-              <visual>
-                  <origin xyz="0 0 0" rpy="${side * -PI/2} 0 0"/>
-                  <geometry>
-                      <mesh filename="file://$(find robot_hardware)/urdf/meshes/Wheel.stl"/>
-                  </geometry>
-                  <material name="black"/>
-              </visual>
-              <!-- INERTIAL -->
-              <inertial>
-                  <origin xyz="0 0 0" rpy="${PI/2} 0 ${PI/2}"/>
-                  <mass value="${wheel_mass}"/>
-                  <inertia
-                      ixx="0.000270" ixy="0.0" ixz="0.0"
-                      iyy="0.000270" iyz="0.0"
-                      izz="0.000426"/>
-              </inertial>
-          </link>
-          <gazebo reference="${name}_wheel">
-              <material>Gazebo/Black</material>
-          </gazebo>
-          <joint name="${name}_wheel_joint" type="continuous">
-              <parent link="${prefix}chassis_link"/>
-              <child link="${name}_wheel"/>
-              <origin xyz="${front * .120} ${side * .129} -.0199" rpy="0 0 0"/>
-              <axis xyz="0 1 0"/>
-              <limit effort="1000.0" velocity="100.0"/>
-              <dynamics damping="${damping}"/>
-              <!-- <mimic joint="${prefix}virtual_rear_wheel_joint" multiplier="1.0" offset="0.0"/> -->
-          </joint>
-      </xacro:macro>
-      <!-- ====================================================================================================== -->
-      <xacro:wheel name="front_left" x="0" y="0" z="0" front="1" side="1"/>
-      <xacro:wheel name="front_right" x="0" y="0" z="0" front="1" side="-1"/>
-      <xacro:wheel name="rear_left" x="0" y="0" z="0" front="-1" side="1"/>
-      <xacro:wheel name="rear_right" x="0" y="0" z="0" front="-1" side="-1"/>
+    <!-- Base Link and Base Footprint -->
+    <xacro:include filename="$(find robot_hardware)/urdf/components/base.xacro" />
+    <!-- Chassis Link -->
+    <xacro:include filename="$(find robot_hardware)/urdf/components/chassis.xacro" />
+        <xacro:include filename="$(find robot_hardware)/urdf/macros/front_wheel.xacro" />
+        <xacro:include filename="$(find robot_hardware)/urdf/macros/rear_wheel.xacro" />
+        <xacro:front_wheel name="front_left" x="${wheel_x}" y="${wheel_y}" z="${wheel_z}" side="1"/>
+        <xacro:front_wheel name="front_right" x="${wheel_x}" y="${-wheel_y}" z="${wheel_z}" side="-1"/>
+        <xacro:rear_wheel name="rear_left" x="${-wheel_x}" y="${wheel_y}" z="${wheel_z}" side="1"/>
+        <xacro:rear_wheel name="rear_right" x="${-wheel_x}" y="${-wheel_y}" z="${wheel_z}" side="-1"/>
   </xacro:macro>
 </robot>

File: ros2_ws/src/robot_hardware/description/urdf/util/constants.xacro (robot description, xacro)
@@ -7,25 +7,15 @@
         <xacro:property name="damping" value="0.001"/>
     <!-- System Wide Constants -->
-        <xacro:property name="base_mass" value="20" /> <!-- arbitrary value for base mass -->
-        <xacro:property name="base_width" value="0.35" />
-        <xacro:property name="base_length" value="0.50" />
-        <xacro:property name="base_height" value="0.25" />
+        <xacro:property name="chassis_mass" value="20" /> <!-- arbitrary value for chassis mass -->
     <!-- Mechanism Specific -->
         <!-- Wheels -->
-            <xacro:property name="wheelbase" value="0.350" />
-            <xacro:property name="wheel_width" value="0.05" />
-            <xacro:property name="wheel_radius" value="0.1" />
+            <xacro:property name="track_width" value="0.165" />
+            <xacro:property name="track_length" value="0.18" />
+            <xacro:property name="wheel_width" value="0.03" />
+            <xacro:property name="wheel_radius" value="0.03725" />
             <xacro:property name="wheel_mass" value="0.5" /> <!-- arbitrary value for wheel mass -->
-            <xacro:property name="front_left_wheel_x" value="0.150"/>
-            <xacro:property name="front_left_wheel_y" value="0.175"/>
-            <xacro:property name="front_left_wheel_z" value="0.00"/>
-            <xacro:property name="front_right_wheel_x" value="0.150"/>
-            <xacro:property name="front_right_wheel_y" value="-0.175"/>
-            <xacro:property name="front_right_wheel_z" value="0.00"/>
-            <xacro:property name="back_left_wheel_x" value="-0.150"/>
-            <xacro:property name="back_left_wheel_y" value="0.175"/>
-            <xacro:property name="back_left_wheel_z" value="0.00"/>
-            <xacro:property name="back_right_wheel_x" value="-0.150"/>
-            <xacro:property name="back_right_wheel_y" value="-0.175"/>
-            <xacro:property name="back_right_wheel_z" value="0.00"/>
+            <!-- Remember to switch X and Y for onshape to ros -->
+            <xacro:property name="wheel_x" value="0.09"/>
+            <xacro:property name="wheel_y" value="0.0675"/>
+            <xacro:property name="wheel_z" value="0.02"/>
 </robot>
