Commit message: Started working on ros2_control xacro

File: ros2_ws/src/robot_hardware/description/ros2_control/robot_hardware.ros2_control.xacro (robot description, xacro)
@@ -8,15 +8,21 @@
             <hardware>
                 <plugin>robot_hardware/RobotSystemHardware</plugin>
+                <!-- For initializing the serial port -->
+                <param name="MCU_field">product</param>
+                <param name="MCU_description">STM32 Virtual ComPort</param>
+                <!-- <param name="my_int_param">0</param> -->
+                <!-- <param name="my_string_param">Hello World</param> -->
             </hardware>
-            <joint name="${prefix}virtual_rear_wheel_joint">
+            <joint name="${prefix}drive_motor">
                 <command_interface name="velocity"/>
-                <state_interface name="velocity"/>
-                <state_interface name="position"/>
+                <!-- RC car doesn't have feedback -->
+                <!-- <state_interface name="velocity"/> -->
+                <!-- <state_interface name="position"/> -->
                 <state_interface name="effort"/>
             </joint>
-            <joint name="${prefix}virtual_front_wheel_joint">
+            <joint name="${prefix}steering_servo">
                 <command_interface name="position"/>
                 <state_interface name="position"/>
-                <state_interface name="effort"/>
+                <!-- <state_interface name="effort"/> -->
             </joint>
         </ros2_control>

Commit message: robot_hardware working

File: ros2_ws/src/robot_hardware/description/ros2_control/robot_hardware.ros2_control.xacro (robot description, xacro)
@@ -3,4 +3,27 @@
 <xacro:macro name="robot_hardware_ros2_control" params="name prefix">
     <xacro:property name="speed_multiplier" value="1"/>
+    <xacro:macro name="front_wheel" params="name">
+        <joint name="${name}_wheel_joint">
+            <command_interface name="velocity"/>
+            <!-- RC car doesn't have feedback -->
+            <!-- <state_interface name="velocity"/> -->
+            <!-- <state_interface name="position"/> -->
+            <!-- <state_interface name="effort"/> -->
+        </joint>
+        <joint name="${name}_steer_joint">
+            <command_interface name="position"/>
+            <!-- <state_interface name="position"/> -->
+            <!-- <state_interface name="effort"/> -->
+        </joint>
+    </xacro:macro>
+    <xacro:macro name="rear_wheel" params="name">
+        <joint name="${name}_wheel_joint">
+            <command_interface name="velocity"/>
+            <!-- RC car doesn't have feedback -->
+            <!-- <state_interface name="velocity"/> -->
+            <!-- <state_interface name="position"/> -->
+            <!-- <state_interface name="effort"/> -->
+        </joint>
+    </xacro:macro>
     <!-- If NOT Sim Mode (Real Mode) -->
     <xacro:unless value="$(arg sim_mode)">
@@ -14,16 +37,8 @@
                 <!-- <param name="my_string_param">Hello World</param> -->
             </hardware>
-            <joint name="${prefix}drive_motor">
-                <command_interface name="velocity"/>
-                <!-- RC car doesn't have feedback -->
-                <!-- <state_interface name="velocity"/> -->
-                <!-- <state_interface name="position"/> -->
-                <state_interface name="effort"/>
-            </joint>
-            <joint name="${prefix}steering_servo">
-                <command_interface name="position"/>
-                <state_interface name="position"/>
-                <!-- <state_interface name="effort"/> -->
-            </joint>
+            <xacro:front_wheel name="${prefix}front_left"/>
+            <xacro:front_wheel name="${prefix}front_right"/>
+            <xacro:rear_wheel name="${prefix}rear_left"/>
+            <xacro:rear_wheel name="${prefix}rear_right"/>
         </ros2_control>
     </xacro:unless>

Commit message: UPdated servo bounds

File: ros2_ws/src/robot_hardware/description/ros2_control/robot_hardware.ros2_control.xacro (robot description, xacro)
@@ -35,8 +35,8 @@
                 <param name="MCU_description">STM32 Virtual ComPort</param>
                 <!-- Servo Bounds (in degrees) -->
-                <param name="Servo_Lower_Bound_Degrees">100</param>
-                <param name="Servo_Upper_Bound_Degrees">170</param>
+                <param name="Servo_Lower_Bound_Degrees">120</param>
+                <param name="Servo_Upper_Bound_Degrees">150</param>
                 <!-- Servo Center Position (in degrees) -->
-                <param name="Servo_Center_Degrees">130</param>
+                <param name="Servo_Center_Degrees">135</param>
                 <!-- <param name="my_int_param">0</param> -->
                 <!-- <param name="my_string_param">Hello World</param> -->

File: ros2_ws/src/robot_hardware/description/urdf/util/constants.xacro (robot description, xacro)
@@ -18,4 +18,4 @@
             <xacro:property name="wheel_x" value="0.09"/>
             <xacro:property name="wheel_y" value="0.0675"/>
-            <xacro:property name="wheel_z" value="0.02"/>
+            <xacro:property name="wheel_z" value="-0.02"/>
 </robot>
